Commit message: docker checkpoint

File: ros2_ws/src/indy7_description/urdf/indy7.urdf (robot description, URDF)
Before this commit: robot indy, 9 links, 8 joints
Links:
- link link0: geometry collision mesh filename=package://indy7_description/meshes/indy7/collision/Indy7_0.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; visual mesh filename=package://indy7_description/meshes/indy7/visual/Indy7_0.stl
- link link1: geometry collision mesh filename=package://indy7_description/meshes/indy7/collision/Indy7_1.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; visual mesh filename=package://indy7_description/meshes/indy7/visual/Indy7_1.stl
- link link2: geometry collision mesh filename=package://indy7_description/meshes/indy7/collision/Indy7_2.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; visual mesh filename=package://indy7_description/meshes/indy7/visual/Indy7_2.stl
- link link3: geometry collision mesh filename=package://indy7_description/meshes/indy7/collision/Indy7_3.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; visual mesh filename=package://indy7_description/meshes/indy7/visual/Indy7_3.stl
- link link4: geometry collision mesh filename=package://indy7_description/meshes/indy7/collision/Indy7_4.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; visual mesh filename=package://indy7_description/meshes/indy7/visual/Indy7_4.stl
- link link5: geometry collision mesh filename=package://indy7_description/meshes/indy7/collision/Indy7_5.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; visual mesh filename=package://indy7_description/meshes/indy7/visual/Indy7_5.stl
- link link6: geometry collision mesh filename=package://indy7_description/meshes/indy7/collision/Indy7_6.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; visual mesh filename=package://indy7_description/meshes/indy7/visual/Indy7_6.stl

Commit message: All the function is completed in the code.

File: ros2_ws/src/indy7_description/urdf/indy7.urdf (robot description, URDF)
Before this commit: robot indy, 9 links, 8 joints
Links:
- added link hand_tcp
Joints:
- added joint hand_tcp_fixed: type fixed, parent tcp, child hand_tcp, origin xyz=-0.1 0 0.08 rpy=0 -3.141592653589793 0
